File: Labs/Hardware/Lab1/Lab1.kicad_pcb (KiCad board)
At the start: 2 copper layers, 40 x 40 mm, 25 parts, among them J1 USB_OTG, J2 Conn_01x06_Male, U1 LM1117ADJ, U2 STM32F411RETx, Y1 8.0MHz

Commit message: Lab2 med gerber
Parts:
- J2: footprint Pin_Headers:Pin_Header_Straight_1x06_Pitch2.54mm_SMD_Pin1Left -> Pin_Headers:Pin_Header_Straight_1x06_Pitch2.54mm
- Y1: footprint Crystals:Crystal_HC49-U_Vertical -> Crystals:Crystal_SMD_HC49-SD_HandSoldering
- moved C1 49.3 mm to (107.9, 94.8), turned to 270 degrees
- moved C6 48.3 mm to (123.9, 86.0), turned to 270 degrees
- moved C8 48.1 mm to (119.5, 86.1), turned to 270 degrees
- moved C9 39.0 mm to (126.1, 85.9), turned to 270 degrees
- moved C11 35.3 mm to (130.4, 73.1)
- moved C15 30.9 mm to (133.4, 77.3), turned to 270 degrees
- moved R1 30.6 mm to (120.4, 65.5), turned to 180 degrees
- moved C16 29.1 mm to (135.9, 94.7)
- moved C14 25.5 mm to (119.1, 68.7), turned to 90 degrees
- moved C12 25.0 mm to (117.2, 68.8), turned to 90 degrees
- moved R4 22.4 mm to (123.1, 89.3)
- moved C7 22.3 mm to (130.8, 95.5), turned to 270 degrees
- moved U1 22.1 mm to (124.9, 95.3)
- moved R3 22.1 mm to (123.1, 91.0)
- moved R2 21.8 mm to (109.8, 80.4), turned to 90 degrees
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Routing:
- net +3V3: track 0.00 -> 122.0 mm, vias 0 -> 5
- net /NRST: track 0.00 -> 44.2 mm
- net /SWO: track 0.00 -> 36.2 mm
- net +5V: track 0.00 -> 24.8 mm
- net /SWCLK: track 0.00 -> 21.7 mm
- net Net-(C2-Pad1): track 0.00 -> 15.4 mm
- net Net-(C5-Pad1): track 0.00 -> 14.9 mm
- net /SWDIO: track 0.00 -> 14.4 mm
- net GND: track 0.00 -> 10.3 mm, vias 0 -> 22
- net Net-(R1-Pad1): track 0.00 -> 6.90 mm
- net Net-(R3-Pad2): track 0.00 -> 3.98 mm
- net Net-(C6-Pad1): track 0.00 -> 1.92 mm
- added copper zone on B.Cu, net GND
Other:
- rule via_min_size: 0.8 -> 0.6
