File: Labs/Hardware/Lab1/Lab1.sch (KiCad schematic (older format))
At the start: 16 parts

Commit message: Lab 1
Parts:
- added C1, C4, C7: 100n, Capacitors_SMD:C_0805_HandSoldering, symbol Device:C
- added C16, C3: 10u, Capacitors_SMD:CP_Elec_5x5.3, symbol Device:CP
- added J1: USB_OTG, Connector_USB:USB_Mini-B_AdamTech_MUSB-B5-S-VT-TSMT-1_SMD_Vertical, symbol Connector:USB_OTG
- added R3: 3,3k, Resistors_SMD:R_0805_HandSoldering, symbol Device:R
- added R4: 5,6k, Resistors_SMD:R_0805_HandSoldering, symbol Device:R
- added U1: LM1117ADJ, TO_SOT_Packages_SMD:SOT-223, symbol E7020E:LM1117ADJ
- C10, C11, C12, C13, C14, C15, C2, C5, C6, C8, C9: renamed from C?; footprint (none) -> Capacitors_SMD:C_0805_HandSoldering
- J2: renamed from J?; footprint (none) -> Pin_Headers:Pin_Header_Straight_1x06_Pitch2.54mm_SMD_Pin1Left
- R1, R2: renamed from R?; footprint (none) -> Resistors_SMD:R_0805_HandSoldering
- U2: renamed from U?; footprint Package_QFP:LQFP-64_10x10mm_P0.5mm -> Housings_QFP:LQFP-64_10x10mm_Pitch0.5mm
- Y1: renamed from Y?; footprint (none) -> Crystals:Crystal_HC49-U_Vertical
Connections:
- net +3V3: now also C10.1, C13.1, U2.13 (VDDA), C16.1, C7.1, R3.1, U1.2 (Vout), U1.4 (Vout2)
- net GND: now also C1.2, C16.2, C3.2, C4.2, C7.2, J1.5 (GND), J1.6 (Shield), R4.2
- net PA0: now reaches U2.14 (PA0)
- net PA1: now reaches U2.15 (PA1)
- new net: R3.2, R4.1, U1.1 (ADJ)
- new net +5V: C1.1, C3.1, C4.1, J1.1 (VBUS), U1.3 (Input)
- new net D+: J1.3 (D+)
- new net D-: J1.2 (D-)
- new net ID: J1.4 (ID)
- no-connect marks 0 -> 49

Commit message: Lab2 med gerber
Parts:
- J2: footprint Pin_Headers:Pin_Header_Straight_1x06_Pitch2.54mm_SMD_Pin1Left -> Pin_Headers:Pin_Header_Straight_1x06_Pitch2.54mm
- Y1: footprint Crystals:Crystal_HC49-U_Vertical -> Crystals:Crystal_SMD_HC49-SD_HandSoldering
Changed lines of the file:
@@
 F 0 "Y1" V 3054 4081 50  0000 L CNN
 F 1 "8.0MHz" V 3145 4081 50  0000 L CNN
-F 2 "Crystals:Crystal_HC49-U_Vertical" H 3100 3950 50  0001 C CNN
+F 2 "Crystals:Crystal_SMD_HC49-SD_HandSoldering" H 3100 3950 50  0001 C CNN
 F 3 "~" H 3100 3950 50  0001 C CNN
 	1    3100 3950
@@
 F 0 "J2" H 8706 4328 50  0000 C CNN
 F 1 "Conn_01x06_Male" H 8706 4237 50  0000 C CNN
-F 2 "Pin_Headers:Pin_Header_Straight_1x06_Pitch2.54mm_SMD_Pin1Left" H 8600 3950 50  0001 C CNN
+F 2 "Pin_Headers:Pin_Header_Straight_1x06_Pitch2.54mm" H 8600 3950 50  0001 C CNN
 F 3 "~" H 8600 3950 50  0001 C CNN
 	1    8600 3950
