File: Labs/Hardware/Lab1/_autosave-Lab1.kicad_pcb (KiCad board)
At the start: 2 copper layers, 40 x 40 mm, 25 parts, among them J1 USB_OTG, J2 Conn_01x06_Male, U1 LM1117ADJ, U2 STM32F411RETx, Y1 8.0MHz

Commit message: Lab2 med gerber
Parts:
- moved J1 1.30 mm to (103.8, 92.0)
- moved C15 1.20 mm to (133.4, 77.3)
- moved C16 1.00 mm to (135.9, 94.7)
- moved C3 0.92 mm to (114.8, 94.1)
- moved J2 0.92 mm to (136.1, 76.0)
- moved C7 0.80 mm to (130.8, 95.5)
- moved U1 0.40 mm to (124.9, 95.3)
- moved R3 0.36 mm to (123.1, 91.0)
- moved R4 0.28 mm to (123.1, 89.3)
Routing:
- net +5V: track 23.2 -> 24.8 mm
- net +3V3: track 120.7 -> 122.0 mm
- net /SWCLK: track 22.3 -> 21.7 mm
- net /SWO: track 36.8 -> 36.2 mm
- net GND: vias 22 -> 21
