File: Project/Hardware/Schematic/lab.sch (KiCad schematic (older format))
At the start: 29 parts, among them J1 USB_B_Micro, J2 6P Male, J3 Conn_01x03_Male, U1 NCP1117-5.0_SOT223, U2 STM32F411RETx, U3 NCP1117-3.3_SOT223, Y1 8MHz

Commit message: Lade till symbol för +7V och 7-voltsregulatorn, samt kopplade in regulatorn.
Parts:
- removed C1, C5: 10u, Capacitor_THT:CP_Radial_D5.0mm_P2.00mm, symbol Device:C_Small
- removed C3, C6: 100n, Capacitor_SMD:C_0805_2012Metric_Pad1.15x1.40mm_HandSolder, symbol Device:C_Small
- removed U1: NCP1117-5.0_SOT223, Package_TO_SOT_SMD:SOT-223-3_TabPin2, symbol Regulator_Linear:NCP1117-5.0_SOT223
- added C? (x2): C, symbol Device:C
- added R? (x2): R, symbol Device:R
- added U?: BD70GC0WEFJ-E2, symbol PASC:BD70GC0WEFJ-E2
Connections:
- net labels added: +7V
- net labels removed: +12V
- wire segments 164 -> 166
Changed lines of the file:
@@
 Text Label 7900 4700 0    50   ~ 0
 SWO
-$Comp
-L Device:C_Small C1
-U 1 1 5C500035
-P 2400 1300
-F 0 "C1" H 2492 1346 50  0000 L CNN
-F 1 "10u" H 2492 1255 50  0000 L CNN
-F 2 "Capacitor_THT:CP_Radial_D5.0mm_P2.00mm" H 2400 1300 50  0001 C CNN
-F 3 "~" H 2400 1300 50  0001 C CNN
-	1    2400 1300
-	1    0    0    -1
-$EndComp
-Wire Wire Line
-	2400 1100 2400 1200
-Connection ~ 2400 1100
-Wire Wire Line
-	2400 1100 2700 1100
-Wire Wire Line
-	2400 1600 2700 1600
-$Comp
-L Device:C_Small C5
-U 1 1 5C514E5C
-P 3900 1300
-F 0 "C5" H 3992 1346 50  0000 L CNN
-F 1 "10u" H 3992 1255 50  0000 L CNN
-F 2 "Capacitor_THT:CP_Radial_D5.0mm_P2.00mm" H 3900 1300 50  0001 C CNN
-F 3 "~" H 3900 1300 50  0001 C CNN
-	1    3900 1300
-	1    0    0    -1
-$EndComp
-Wire Wire Line
-	3900 1100 3900 1200
-Wire Wire Line
-	3900 1400 3900 1600
-$Comp
-L Device:C_Small C6
-U 1 1 5C51CB4F
-P 4200 1300
-F 0 "C6" H 4292 1346 50  0000 L CNN
-F 1 "100n" H 4292 1255 50  0000 L CNN
-F 2 "Capacitor_SMD:C_0805_2012Metric_Pad1.15x1.40mm_HandSolder" H 4200 1300 50  0001 C CNN
-F 3 "~" H 4200 1300 50  0001 C CNN
-	1    4200 1300
-	1    0    0    -1
-$EndComp
-$Comp
-L Device:C_Small C3
-U 1 1 5C51F65E
-P 2700 1300
-F 0 "C3" H 2792 1346 50  0000 L CNN
-F 1 "100n" H 2792 1255 50  0000 L CNN
-F 2 "Capacitor_SMD:C_0805_2012Metric_Pad1.15x1.40mm_HandSolder" H 2700 1300 50  0001 C CNN
-F 3 "~" H 2700 1300 50  0001 C CNN
-	1    2700 1300
-	1    0    0    -1
-$EndComp
-Wire Wire Line
-	2700 1200 2700 1100
-Wire Wire Line
-	2700 1400 2700 1600
-Wire Wire Line
-	3900 1100 4200 1100
-Wire Wire Line
-	4200 1100 4200 1200
-Wire Wire Line
-	4200 1400 4200 1600
-Wire Wire Line
-	4200 1600 3900 1600
-Wire Wire Line
-	2400 900  2400 1100
 Text Label 3200 4300 0    50   ~ 0
 SWCLK
@@
 Wire Wire Line
 	3600 4600 4100 4600
-$Comp
-L power:GND #PWR0114
-U 1 1 5C56D6CB
-P 3300 1700
-F 0 "#PWR0114" H 3300 1450 50  0001 C CNN
-F 1 "GND" H 3305 1527 50  0000 C CNN
-F 2 "" H 3300 1700 50  0001 C CNN
-F 3 "" H 3300 1700 50  0001 C CNN
-	1    3300 1700
-	1    0    0    -1
-$EndComp
-Wire Wire Line
-	4200 1100 4200 900
-Connection ~ 4200 1100
 NoConn ~ 7500 2900
 NoConn ~ 7500 3000
@@
 Connection ~ 4200 2700
 $Comp
-L Regulator_Linear:NCP1117-5.0_SOT223 U1
-U 1 1 5C5D36EE
-P 3300 1100
-F 0 "U1" H 3300 1342 50  0000 C CNN
-F 1 "NCP1117-5.0_SOT223" H 3300 1251 50  0000 C CNN
-F 2 "Package_TO_SOT_SMD:SOT-223-3_TabPin2" H 3300 1300 50  0001 C CNN
-F 3 "http://www.onsemi.com/pub_link/Collateral/NCP1117-D.PDF" H 3400 850 50  0001 C CNN
-	1    3300 1100
-	1    0    0    -1
-$EndComp
-$Comp
 L Regulator_Linear:NCP1117-3.3_SOT223 U3
 U 1 1 5C5D379C
@@
 	1    0    0    -1
 $EndComp
-$Comp
-L power:+BATT #PWR0111
-U 1 1 5C5D3900
-P 2400 900
-F 0 "#PWR0111" H 2400 750 50  0001 C CNN
-F 1 "+BATT" H 2415 1073 50  0000 C CNN
-F 2 "" H 2400 900 50  0001 C CNN
-F 3 "" H 2400 900 50  0001 C CNN
-	1    2400 900
-	1    0    0    -1
-$EndComp
-Wire Wire Line
-	2700 1100 3000 1100
-Connection ~ 2700 1100
-Wire Wire Line
-	3600 1100 3900 1100
-Connection ~ 3900 1100
-Wire Wire Line
-	3900 1600 3300 1600
-Wire Wire Line
-	3300 1600 3300 1700
-Connection ~ 3900 1600
-Wire Wire Line
-	3300 1600 2700 1600
-Connection ~ 3300 1600
-Connection ~ 2700 1600
-Wire Wire Line
-	2400 1600 2400 1400
-Wire Wire Line
-	3300 1400 3300 1600
 Wire Wire Line
 	2700 2700 3000 2700
@@
 	9250 5200 9650 5200
 $Comp
-L power:+12V #PWR?
-U 1 1 5C679F70
-P 4200 900
-F 0 "#PWR?" H 4200 750 50  0001 C CNN
-F 1 "+12V" H 4215 1073 50  0000 C CNN
-F 2 "" H 4200 900 50  0001 C CNN
-F 3 "" H 4200 900 50  0001 C CNN
-	1    4200 900
-	1    0    0    -1
-$EndComp
+L PASC:BD70GC0WEFJ-E2 U?
+U 1 1 5C5F4321
+P 3200 1200
+F 0 "U?" H 3200 1565 50  0000 C CNN
+F 1 "BD70GC0WEFJ-E2" H 3200 1474 50  0000 C CNN
+F 2 "" H 2600 1800 50  0001 C CNN
+F 3 "" H 2600 1800 50  0001 C CNN
+	1    3200 1200
+	1    0    0    -1
+$EndComp
+Wire Wire Line
+	2700 1200 2600 1200
+Wire Wire Line
+	2600 1200 2600 1100
+Wire Wire Line
+	2600 1100 2700 1100
+$Comp
+L Device:C C?
+U 1 1 5C6012C4
+P 2400 1400
+F 0 "C?" H 2515 1446 50  0000 L CNN
+F 1 "C" H 2515 1355 50  0000 L CNN
+F 2 "" H 2438 1250 50  0001 C CNN
+F 3 "~" H 2400 1400 50  0001 C CNN
+	1    2400 1400
+	1    0    0    -1
+$EndComp
+Wire Wire Line
+	2400 1250 2400 1100
+Wire Wire Line
+	2400 1100 2600 1100
+Connection ~ 2600 1100
+$Comp
+L Device:R R?
+U 1 1 5C615406
+P 3400 1700
+F 0 "R?" V 3300 1650 50  0000 C CNN
+F 1 "R" V 3225 1675 50  0000 C CNN
+F 2 "" V 3330 1700 50  0001 C CNN
+F 3 "~" H 3400 1700 50  0001 C CNN
+	1    3400 1700
+	0    -1   -1   0
+$EndComp
+$Comp
+L Device:C C?
+U 1 1 5C6157A1
+P 4400 1400
+F 0 "C?" H 4515 1446 50  0000 L CNN
+F 1 "C" H 4515 1355 50  0000 L CNN
+F 2 "" H 4438 1250 50  0001 C CNN
+F 3 "~" H 4400 1400 50  0001 C CNN
+	1    4400 1400
+	1    0    0    -1
+$EndComp
+Wire Wire Line
+	4400 1250 4400 1100
+Wire Wire Line
+	3250 1700 3100 1700
+Wire Wire Line
+	4000 1550 4000 1700
+Wire Wire Line
+	3550 1700 3800 1700
+Wire Wire Line
+	3700 1100 4000 1100
+$Comp
+L Device:R R?
+U 1 1 5C6153A2
+P 4000 1400
+F 0 "R?" H 4070 1446 50  0000 L CNN
+F 1 "R" H 4070 1355 50  0000 L CNN
+F 2 "" V 3930 1400 50  0001 C CNN
+F 3 "~" H 4000 1400 50  0001 C CNN
+	1    4000 1400
+	1    0    0    -1
+$EndComp
+Wire Wire Line
+	4000 1250 4000 1100
+Connection ~ 4000 1100
+Wire Wire Line
+	4400 1100 4000 1100
+Wire Wire Line
+	3100 1700 3100 1500
+Wire Wire Line
+	3800 1700 3800 1200
+Wire Wire Line
+	3800 1200 3700 1200
+Connection ~ 3800 1700
+Wire Wire Line
+	3800 1700 4000 1700
+$Comp
+L power:GND #PWR?
+U 1 1 5C6BBC5B
+P 3100 1800
+F 0 "#PWR?" H 3100 1550 50  0001 C CNN
+F 1 "GND" H 3105 1627 50  0000 C CNN
+F 2 "" H 3100 1800 50  0001 C CNN
+F 3 "" H 3100 1800 50  0001 C CNN
+	1    3100 1800
+	1    0    0    -1
+$EndComp
+Wire Wire Line
+	3100 1800 3100 1700
+Connection ~ 3100 1700
+Wire Wire Line
+	2400 1700 3100 1700
+Wire Wire Line
+	2400 1550 2400 1700
+$Comp
+L power:GND #PWR?
+U 1 1 5C6D4879
+P 4400 1800
+F 0 "#PWR?" H 4400 1550 50  0001 C CNN
+F 1 "GND" H 4405 1627 50  0000 C CNN
+F 2 "" H 4400 1800 50  0001 C CNN
+F 3 "" H 4400 1800 50  0001 C CNN
+	1    4400 1800
+	1    0    0    -1
+$EndComp
+Wire Wire Line
+	4400 1550 4400 1800
+$Comp
+L PASC:+7V #PWR?
+U 1 1 5C6FF278
+P 4400 900
+F 0 "#PWR?" H 4650 1000 50  0001 C CNN
+F 1 "+7V" H 4385 1074 50  0000 C CNN
+F 2 "" H 4400 900 50  0001 C CNN
+F 3 "" H 4400 900 50  0001 C CNN
+	1    4400 900
+	1    0    0    -1
+$EndComp
+Wire Wire Line
+	4400 1100 4400 900
+Connection ~ 4400 1100
+$Comp
+L power:+BATT #PWR?
+U 1 1 5C7205D7
+P 2400 900
+F 0 "#PWR?" H 2400 750 50  0001 C CNN
+F 1 "+BATT" H 2415 1073 50  0000 C CNN
+F 2 "" H 2400 900 50  0001 C CNN
+F 3 "" H 2400 900 50  0001 C CNN
+	1    2400 900
+	1    0    0    -1
+$EndComp
+Wire Wire Line
+	2400 900  2400 1100
+Connection ~ 2400 1100
 $EndSCHEMATC
