File: Project/Hardware/Schematic/tempsensor.sch (KiCad schematic (older format))
At the start: 12 parts

Commit message: Fixa bibliotek ref
Parts:
- U?: symbol lab-rescue:MAX4460ESA+-PASC -> PASC:MAX4460ESA+
Changed lines of the file:
@@
 $EndComp
 $Comp
-L lab-rescue:MAX4460ESA+-PASC U?
+L PASC:MAX4460ESA+ U?
 U 1 1 5C562619
 P 5000 2100
