File: Project/Hardware/Schematic_Ubuntu/lab.kicad_pcb (KiCad board)
At the start: 2 copper layers, 56 parts, among them J1 USB_B_Micro, J2 6P Male, J3 Conn_01x03_Male, Q1 2N3904, SW1 SW_SPDT, U1 NCP1117-3.3_SOT223, U10 MomentSwitch, U11 MomentSwitch, U2 STM32F411RETx, U3 lis3dh_board, U4 Pulse_sensor, U5 MAX4460ESA+, U6 Nokia5110, U7 piezo, U8 MomentSwitch, U9 MomentSwitch, Y1 8MHz

Commit message: Missade några filer förra commiten
Parts:
- moved SW1 22.9 mm to (78.0, 104.0), turned to 90 degrees
Changed lines of the file:
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@@
-(kicad_pcb (version 20171130) (host pcbnew 5.0.2-bee76a0~70~ubuntu16.04.1)
+(kicad_pcb (version 20171130) (host pcbnew "(5.0.2)-1")
   (general
     (thickness 1.6)
-    (drawings 0)
+    (drawings 3)
     (tracks 74)
     (zones 0)
@@
     (solder_mask_min_width 0.25)
     (aux_axis_origin 0 0)
-    (visible_elements FFFFFF7F)
+    (visible_elements 7FFFFFFF)
     (pcbplotparams
       (layerselection 0x010fc_ffffffff)
@@
       (effects (font (size 1 1) (thickness 0.15)))
     )
-    (fp_line (start -10 10) (end -10 0) (layer F.SilkS) (width 0.15))
-    (fp_line (start 10 10) (end -10 10) (layer F.SilkS) (width 0.15))
-    (fp_line (start 10 -10) (end 10 10) (layer F.SilkS) (width 0.15))
-    (fp_line (start -10 -10) (end 10 -10) (layer F.SilkS) (width 0.15))
-    (fp_line (start -10 0) (end -10 -10) (layer F.SilkS) (width 0.15))
-    (pad 11 thru_hole circle (at 3.81 -4.92) (size 1.5 1.5) (drill 1) (layers *.Cu *.Mask))
-    (pad 10 thru_hole circle (at 1.27 -4.91) (size 1.5 1.5) (drill 1) (layers *.Cu *.Mask))
-    (pad 9 thru_hole circle (at -1.27 -4.92) (size 1.5 1.5) (drill 1) (layers *.Cu *.Mask))
-    (pad 8 thru_hole circle (at 8.89 7.46) (size 1.5 1.5) (drill 1) (layers *.Cu *.Mask)
+    (fp_line (start -10.16 10.16) (end -10.16 -10.16) (layer F.SilkS) (width 0.15))
+    (fp_line (start -10.16 -10.16) (end 10.16 -10.16) (layer F.SilkS) (width 0.15))
+    (fp_line (start 10.16 -10.16) (end 10.16 10.16) (layer F.SilkS) (width 0.15))
+    (fp_line (start 10.16 10.16) (end -10.16 10.16) (layer F.SilkS) (width 0.15))
+    (pad "" thru_hole circle (at -7.62 -7.62) (size 3.5 3.5) (drill 2.54) (layers *.Cu *.Mask))
+    (pad "" thru_hole circle (at 7.62 -7.62) (size 3.5 3.5) (drill 2.54) (layers *.Cu *.Mask))
+    (pad 1 thru_hole rect (at -8.89 7.62) (size 1.5 1.5) (drill 1) (layers *.Cu *.Mask)
+      (net 10 +3V3))
+    (pad 2 thru_hole circle (at -6.35 7.62) (size 1.5 1.5) (drill 1) (layers *.Cu *.Mask)
+      (net 17 "Net-(U3-Pad2)"))
+    (pad 3 thru_hole circle (at -3.81 7.62) (size 1.5 1.5) (drill 1) (layers *.Cu *.Mask)
+      (net 3 GND))
+    (pad 4 thru_hole circle (at -1.27 7.62) (size 1.5 1.5) (drill 1) (layers *.Cu *.Mask)
+      (net 18 /I2C1_SCL))
+    (pad 5 thru_hole circle (at 1.27 7.62) (size 1.5 1.5) (drill 1) (layers *.Cu *.Mask)
+      (net 19 /I2C1_SDA))
+    (pad 6 thru_hole circle (at 3.81 7.62) (size 1.5 1.5) (drill 1) (layers *.Cu *.Mask)
+      (net 3 GND))
+    (pad 7 thru_hole circle (at 6.35 7.62) (size 1.5 1.5) (drill 1) (layers *.Cu *.Mask)
+      (net 10 +3V3))
+    (pad 8 thru_hole circle (at 8.89 7.62) (size 1.5 1.5) (drill 1) (layers *.Cu *.Mask)
       (net 20 /CS_INT))
-    (pad 7 thru_hole circle (at 6.35 7.46) (size 1.5 1.5) (drill 1) (layers *.Cu *.Mask)
-      (net 10 +3V3))
-    (pad 6 thru_hole circle (at 3.81 7.46) (size 1.5 1.5) (drill 1) (layers *.Cu *.Mask)
-      (net 3 GND))
-    (pad 5 thru_hole circle (at 1.27 7.46) (size 1.5 1.5) (drill 1) (layers *.Cu *.Mask)
-      (net 19 /I2C1_SDA))
-    (pad 4 thru_hole circle (at -1.27 7.46) (size 1.5 1.5) (drill 1) (layers *.Cu *.Mask)
-      (net 18 /I2C1_SCL))
-    (pad 3 thru_hole circle (at -3.81 7.46) (size 1.5 1.5) (drill 1) (layers *.Cu *.Mask)
-      (net 3 GND))
-    (pad 2 thru_hole circle (at -6.35 7.46) (size 1.5 1.5) (drill 1) (layers *.Cu *.Mask)
-      (net 17 "Net-(U3-Pad2)"))
-    (pad 1 thru_hole rect (at -8.89 7.46) (size 1.5 1.5) (drill 1) (layers *.Cu *.Mask)
-      (net 10 +3V3))
-    (pad "" thru_hole circle (at 7.5 -7.5) (size 3.5 3.5) (drill 2.54) (layers *.Cu *.Mask))
-    (pad "" thru_hole circle (at -7.5 -7.5) (size 3.5 3.5) (drill 2.54) (layers *.Cu *.Mask))
+    (pad 9 thru_hole circle (at -1.27 -5.08) (size 1.5 1.5) (drill 1) (layers *.Cu *.Mask))
+    (pad 10 thru_hole circle (at 1.27 -5.08) (size 1.5 1.5) (drill 1) (layers *.Cu *.Mask))
+    (pad 11 thru_hole circle (at 3.81 -5.08) (size 1.5 1.5) (drill 1) (layers *.Cu *.Mask))
   )
   (module Pin_Headers:Pin_Header_Straight_1x02_Pitch2.54mm (layer F.Cu)
@@
   )
   (module PASC:SPDT-100 (layer F.Cu)
-    (at 99.9 97.4)
-    (fp_text reference SW1 (at 0.25 7.5) (layer F.SilkS)
-      (effects (font (size 1 1) (thickness 0.15)))
-    )
-    (fp_text value SW_SPDT (at -0.25 -7) (layer F.Fab)
+    (at 78 104 90)
+    (fp_text reference SW1 (at 0.25 7.5 90) (layer F.SilkS)
+      (effects (font (size 1 1) (thickness 0.15)))
+    )
+    (fp_text value SW_SPDT (at -0.25 -7 90) (layer F.Fab)
       (effects (font (size 1 1) (thickness 0.15)))
     )
@@
     (fp_line (start 6.85 -3.3) (end -6.85 -3.3) (layer F.SilkS) (width 0.15))
     (fp_line (start 6.85 3.3) (end 6.85 -3.3) (layer F.SilkS) (width 0.15))
-    (pad 1 thru_hole circle (at -4.7 0) (size 2.8 2.8) (drill 1.85) (layers *.Cu *.Mask)
+    (pad 1 thru_hole circle (at -4.7 0 90) (size 2.8 2.8) (drill 1.85) (layers *.Cu *.Mask)
       (net 14 +BATT))
-    (pad 2 thru_hole rect (at 0 0) (size 2.8 2.8) (drill 1.85) (layers *.Cu *.Mask)
+    (pad 2 thru_hole rect (at 0 0 90) (size 2.8 2.8) (drill 1.85) (layers *.Cu *.Mask)
       (net 15 +VIN))
-    (pad 3 thru_hole circle (at 4.7 0) (size 2.8 2.8) (drill 1.85) (layers *.Cu *.Mask)
+    (pad 3 thru_hole circle (at 4.7 0 90) (size 2.8 2.8) (drill 1.85) (layers *.Cu *.Mask)
       (net 5 +5V))
   )
@@
     )
   )
+  (dimension 50 (width 0.3) (layer F.SilkS)
+    (gr_text "50.000 mm" (at 217.1 87 90) (layer F.SilkS)
+      (effects (font (size 1.5 1.5) (thickness 0.3)))
+    )
+    (feature1 (pts (xy 206 62) (xy 215.586421 62)))
+    (feature2 (pts (xy 206 112) (xy 215.586421 112)))
+    (crossbar (pts (xy 215 112) (xy 215 62)))
+    (arrow1a (pts (xy 215 62) (xy 215.586421 63.126504)))
+    (arrow1b (pts (xy 215 62) (xy 214.413579 63.126504)))
+    (arrow2a (pts (xy 215 112) (xy 215.586421 110.873496)))
+    (arrow2b (pts (xy 215 112) (xy 214.413579 110.873496)))
+  )
+  (dimension 60 (width 0.3) (layer F.SilkS)
+    (gr_text "60.000 mm" (at 200.1 82 90) (layer F.SilkS)
+      (effects (font (size 1.5 1.5) (thickness 0.3)))
+    )
+    (feature1 (pts (xy 187 52) (xy 198.586421 52)))
+    (feature2 (pts (xy 187 112) (xy 198.586421 112)))
+    (crossbar (pts (xy 198 112) (xy 198 52)))
+    (arrow1a (pts (xy 198 52) (xy 198.586421 53.126504)))
+    (arrow1b (pts (xy 198 52) (xy 197.413579 53.126504)))
+    (arrow2a (pts (xy 198 112) (xy 198.586421 110.873496)))
+    (arrow2b (pts (xy 198 112) (xy 197.413579 110.873496)))
+  )
+  (dimension 100 (width 0.3) (layer F.SilkS)
+    (gr_text "100.000 mm" (at 120 136.1) (layer F.SilkS)
+      (effects (font (size 1.5 1.5) (thickness 0.3)))
+    )
+    (feature1 (pts (xy 170 122) (xy 170 134.586421)))
+    (feature2 (pts (xy 70 122) (xy 70 134.586421)))
+    (crossbar (pts (xy 70 134) (xy 170 134)))
+    (arrow1a (pts (xy 170 134) (xy 168.873496 134.586421)))
+    (arrow1b (pts (xy 170 134) (xy 168.873496 133.413579)))
+    (arrow2a (pts (xy 70 134) (xy 71.126504 134.586421)))
+    (arrow2b (pts (xy 70 134) (xy 71.126504 133.413579)))
+  )
   (segment (start 135.1 89.15) (end 135.45 88.8) (width 0.2) (layer F.Cu) (net 7))
