File: Project/Hardware/Schematic_Ubuntu/lab.kicad_pcb (KiCad board)
At the start: 2 copper layers, 87.8 x 48.1 mm, 58 parts, among them J1 USB_B_Micro, J2 6P Male, J3 Conn_01x03_Male, Q1 2N3904, SW1 SW_SPDT, U1 NCP1117-3.3_SOT223, U10 MomentSwitch, U11 MomentSwitch, U2 STM32F411RETx, U3 lis3dh_board, U4 Pulse_sensor, U5 MAX4460ESA+, U6 Nokia5110, U7 piezo, U8 MomentSwitch, U9 MomentSwitch, Y1 8MHz

Commit message: Gerber, csv boom, cap till knappar
Parts:
- added C20: C, Capacitors_SMD:C_0805_HandSoldering, F.Cu at (166.4, 57.1)
- added C21: C, Capacitors_SMD:C_0805_HandSoldering, F.Cu at (166.3, 63.9)
- added C22: C, Capacitors_SMD:C_0805_HandSoldering, F.Cu at (166.3, 70.3)
- moved R17 0.55 mm to (168.1, 70.4)
Routing:
- net /TIM_INC: track 39.1 -> 41.0 mm
- net /TIM_RES: track 33.9 -> 35.8 mm
- net /TIM_START: track 51.4 -> 53.2 mm
- net GND: vias 180 -> 178
Other:
- outline, holes or cut-outs redrawn
