File: Project/Hardware/Schematic_Ubuntu/pcb_rev2.kicad_pcb (KiCad board)
At the start: 2 copper layers, 56 parts, among them J1 USB_B_Micro, J2 6P Male, J3 Conn_01x03_Male, Q1 2N3904, SW1 SW_SPDT, U1 NCP1117-3.3_SOT223, U10 MomentSwitch, U11 MomentSwitch, U2 STM32F411RETx, U3 lis3dh_board, U4 Pulse_sensor, U5 MAX4460ESA+, U6 Nokia5110, U7 piezo, U8 MomentSwitch, U9 MomentSwitch, Y1 8MHz

Commit message: Rev 2 pcb
Parts:
- moved Y1 54.1 mm to (174.6, 108.4), turned to 270 degrees
- moved R4 53.3 mm to (108.2, 102.1), turned to 90 degrees
- moved TH1 53.1 mm to (100.8, 96.0)
- moved R8 50.4 mm to (106.2, 102.1), turned to 90 degrees
- moved C18 50.0 mm to (108.2, 98.6)
- moved R6 48.9 mm to (110.2, 102.1), turned to 90 degrees
- moved C8 48.3 mm to (166.0, 116.9), turned to 270 degrees
- moved U5 47.1 mm to (105.9, 94.7), turned to 270 degrees
- moved C13 46.8 mm to (164.2, 116.9), turned to 270 degrees
- moved C6 46.1 mm to (169.4, 110.7), turned to 270 degrees
- moved R7 46.0 mm to (105.9, 88.1), turned to 90 degrees
- moved Q1 45.9 mm to (95.3, 75.7), turned to 0 degrees
- moved R9 44.0 mm to (108.7, 94.7), turned to 270 degrees
- moved R1 43.8 mm to (161.3, 117.0), turned to 270 degrees
- moved C7 43.3 mm to (169.4, 106.4), turned to 90 degrees
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Routing:
- net +3V3: track 304.2 -> 34.8 mm
- net /SWO: track 49.9 -> 0.00 mm
- net +VIN: track 48.1 -> 0.00 mm
- net /TIM_RES: track 0.00 -> 40.3 mm, vias 0 -> 2
- net /I2C1_SCL: track 19.6 -> 58.4 mm
- net /SWCLK: track 35.2 -> 0.00 mm
- net /SWDIO: track 43.4 -> 8.81 mm
- net /I2C1_SDA: track 24.0 -> 52.8 mm
- net /TIM3_CH1: track 0.00 -> 27.6 mm, vias 0 -> 2
- net /PIEZOPWM: track 24.7 -> 0.00 mm, vias 2 -> 0
- net /CS_INT: track 28.6 -> 53.3 mm
- net +5V: track 24.3 -> 0.00 mm
- net +BATT: track 18.7 -> 0.00 mm
- net /NRST: track 57.6 -> 40.0 mm
- net Net-(D1-Pad2): track 15.5 -> 0.00 mm
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