File: Project/Hardware/Schematic_ons/display.sch (KiCad schematic (older format))
At the start: 3 parts, among them U6 Nokia5110

Commit message: Add files via upload
Added resistor to pulse, and capacitors to buttons
Parts:
- C19: symbol Device:C -> PCB_Simon_mount_rev2-rescue:C-Device
- R12: symbol Device:R -> PCB_Simon_mount_rev2-rescue:R-Device
Changed lines of the file:
@@
 EESchema Schematic File Version 4
+LIBS:PCB_Simon_mount_rev2-cache
 EELAYER 26 0
 EELAYER END
@@
 $EndDescr
 $Comp
-L power:GND #PWR0134
+L PCB_Simon_mount_rev2-rescue:GND-power #PWR0134
 U 1 1 5C58DE2B
 P 1450 1900
@@
 $EndComp
 $Comp
-L Device:C C19
+L PCB_Simon_mount_rev2-rescue:C-Device C19
 U 1 1 5C58DF2A
 P 1450 1600
@@
 LCD_VSS
 $Comp
-L power:+3.3V #PWR0135
+L PCB_Simon_mount_rev2-rescue:+3.3V-power #PWR0135
 U 1 1 5C66DBDE
 P 1450 1300
@@
 LCD_VDD
 $Comp
-L Device:R R12
+L PCB_Simon_mount_rev2-rescue:R-Device R12
 U 1 1 5C63A8F8
 P 2300 1800
@@
 LCD_LED
 $Comp
-L power:GND #PWR0136
+L PCB_Simon_mount_rev2-rescue:GND-power #PWR0136
 U 1 1 5C63AC65
 P 4050 2200
