File: Project/Hardware/Schematic_ons/tempsensor.sch (KiCad schematic (older format))
At the start: 12 parts, among them U5 MAX4460ESA+

Commit message: Add files via upload
Added resistor to pulse, and capacitors to buttons
Parts:
- C18: symbol Device:C -> PCB_Simon_mount_rev2-rescue:C-Device
- R10, R11, R3, R4, R5, R6, R7, R8, R9: symbol Device:R -> PCB_Simon_mount_rev2-rescue:R-Device
- TH1: symbol Sensor_Temperature:PT1000 -> PCB_Simon_mount_rev2-rescue:PT1000-Sensor_Temperature
Changed lines of the file:
@@
 EESchema Schematic File Version 4
+LIBS:PCB_Simon_mount_rev2-cache
 EELAYER 26 0
 EELAYER END
@@
 $EndDescr
 $Comp
-L Sensor_Temperature:PT1000 TH1
+L PCB_Simon_mount_rev2-rescue:PT1000-Sensor_Temperature TH1
 U 1 1 5C561FEF
 P 2700 2000
@@
 $EndComp
 $Comp
-L Device:R R7
+L PCB_Simon_mount_rev2-rescue:R-Device R7
 U 1 1 5C5621D5
 P 2700 1600
@@
 $EndComp
 $Comp
-L Device:R R3
+L PCB_Simon_mount_rev2-rescue:R-Device R3
 U 1 1 5C5622D1
 P 1400 2000
@@
 $EndComp
 $Comp
-L Device:R R8
+L PCB_Simon_mount_rev2-rescue:R-Device R8
 U 1 1 5C562312
 P 2700 2600
@@
 $EndComp
 $Comp
-L Device:R R4
+L PCB_Simon_mount_rev2-rescue:R-Device R4
 U 1 1 5C56234C
 P 1400 2600
@@
 $EndComp
 $Comp
-L power:+3V3 #PWR0128
+L PCB_Simon_mount_rev2-rescue:+3V3-power #PWR0128
 U 1 1 5C5626CF
 P 1100 2100
@@
 	2700 1750 2700 1850
 $Comp
-L power:GND #PWR0129
+L PCB_Simon_mount_rev2-rescue:GND-power #PWR0129
 U 1 1 5C562A08
 P 3100 2450
@@
 INAMPFB
 $Comp
-L Device:R R9
+L PCB_Simon_mount_rev2-rescue:R-Device R9
 U 1 1 5C5639FE
 P 4100 3100
@@
 $EndComp
 $Comp
-L Device:R R10
+L PCB_Simon_mount_rev2-rescue:R-Device R10
 U 1 1 5C563A36
 P 4100 3500
@@
 TEMPOUT
 $Comp
-L power:GND #PWR0130
+L PCB_Simon_mount_rev2-rescue:GND-power #PWR0130
 U 1 1 5C5640C7
 P 4100 4150
@@
 	3900 4500 3900 2700
 $Comp
-L power:+3V3 #PWR0131
+L PCB_Simon_mount_rev2-rescue:+3V3-power #PWR0131
 U 1 1 5C56452F
 P 7200 1400
@@
 	7200 1600 6700 1600
 $Comp
-L power:GND #PWR0132
+L PCB_Simon_mount_rev2-rescue:GND-power #PWR0132
 U 1 1 5C564858
 P 4000 1800
@@
 Wheatstone Bridge for Pt1000 thermistor.\n
 $Comp
-L Device:C C18
+L PCB_Simon_mount_rev2-rescue:C-Device C18
 U 1 1 5C565EBC
 P 7200 1900
@@
 Connection ~ 7200 1600
 $Comp
-L power:GND #PWR0133
+L PCB_Simon_mount_rev2-rescue:GND-power #PWR0133
 U 1 1 5C5665E0
 P 7200 2200
@@
 	3700 3100 3700 800
 $Comp
-L Device:R R5
+L PCB_Simon_mount_rev2-rescue:R-Device R5
 U 1 1 5C58B777
 P 1800 2000
@@
 $EndComp
 $Comp
-L Device:R R6
+L PCB_Simon_mount_rev2-rescue:R-Device R6
 U 1 1 5C58B7A7
 P 1800 2600
@@
 $EndComp
 $Comp
-L Device:R R11
+L PCB_Simon_mount_rev2-rescue:R-Device R11
 U 1 1 5C58C2D0
 P 4100 3900
