File: Project/Hardware/Schematic_ons/accelerometer.sch (KiCad schematic (older format))
At the start: 2 parts, among them U3 lis3dh_board

Commit message: Pcb rev1 simon (#14)
Klar PCB av Simon
Added resistor to pulse, and capacitors to buttons
Parts:
- C16: symbol Device:C -> PCB_Simon_mount_rev2-rescue:C-Device
Changed lines of the file:
@@
 EESchema Schematic File Version 4
-LIBS:lab-cache
+LIBS:PCB_Simon_mount_rev2-cache
 EELAYER 26 0
 EELAYER END
@@
 $EndDescr
 $Comp
-L power:+3.3V #PWR0120
+L PCB_Simon_mount_rev2-rescue:+3.3V-power #PWR0120
 U 1 1 5C5AB0A3
 P 1300 1850
@@
 	1800 2050 1300 2050
 $Comp
-L power:GND #PWR0121
+L PCB_Simon_mount_rev2-rescue:GND-power #PWR0121
 U 1 1 5C59F3FC
 P 2300 2850
@@
 	2300 2750 2300 2850
 $Comp
-L power:GND #PWR0122
+L PCB_Simon_mount_rev2-rescue:GND-power #PWR0122
 U 1 1 5C59F76F
 P 4100 2500
@@
 NoConn ~ 1800 2200
 $Comp
-L Device:C C16
+L PCB_Simon_mount_rev2-rescue:C-Device C16
 U 1 1 5C5A61DB
 P 1300 2350
@@
 $EndComp
 $Comp
-L power:GND #PWR0123
+L PCB_Simon_mount_rev2-rescue:GND-power #PWR0123
 U 1 1 5C5A62A1
 P 1300 2650
@@
 CS_XL
 $Comp
-L power:+3V3 #PWR0124
+L PCB_Simon_mount_rev2-rescue:+3V3-power #PWR0124
 U 1 1 5C5D1727
 P 4100 1900
