File: Project/Hardware/Schematic_ons/piezo.sch (KiCad schematic (older format))
At the start: 5 parts, among them Q1 2N3904, U7 piezo

Commit message: Pcb rev1 simon (#14)
Klar PCB av Simon
Added resistor to pulse, and capacitors to buttons
Parts:
- D1: symbol Diode:1N4148 -> PCB_Simon_mount_rev2-rescue:1N4148-Diode
- Q1: symbol Transistor_BJT:2N3904 -> PCB_Simon_mount_rev2-rescue:2N3904-Transistor_BJT
- R13, R14: symbol Device:R -> PCB_Simon_mount_rev2-rescue:R-Device
Changed lines of the file:
@@
 EESchema Schematic File Version 4
-LIBS:lab-cache
+LIBS:PCB_Simon_mount_rev2-cache
 EELAYER 26 0
 EELAYER END
@@
 $EndComp
 $Comp
-L Device:R R14
+L PCB_Simon_mount_rev2-rescue:R-Device R14
 U 1 1 5C5EB38A
 P 2900 1600
@@
 $EndComp
 $Comp
-L Diode:1N4148 D1
+L PCB_Simon_mount_rev2-rescue:1N4148-Diode D1
 U 1 1 5C5EB4E1
 P 2900 2050
@@
 	2900 2300 2900 2500
 $Comp
-L Device:R R13
+L PCB_Simon_mount_rev2-rescue:R-Device R13
 U 1 1 5C5EB823
 P 2100 2700
@@
 	2250 2700 2600 2700
 $Comp
-L power:GND #PWR0137
+L PCB_Simon_mount_rev2-rescue:GND-power #PWR0137
 U 1 1 5C5EB928
 P 2900 3150
@@
 PIEZOPWM
 $Comp
-L power:+3.3V #PWR0138
+L PCB_Simon_mount_rev2-rescue:+3.3V-power #PWR0138
 U 1 1 5C6DC10D
 P 2900 1100
@@
 $EndComp
 $Comp
-L Transistor_BJT:2N3904 Q1
+L PCB_Simon_mount_rev2-rescue:2N3904-Transistor_BJT Q1
 U 1 1 5C64EC5C
 P 2800 2700
