File: Project/Hardware/Schematic_ons/PCB_Simon_mount_rev2.kicad_pcb (KiCad board)
At the start: 2 copper layers, 80.5 x 53.8 mm, 56 parts, among them J1 USB_B_Micro, J2 6P Male, J3 Conn_01x03_Male, Q1 2N3904, SW1 SW_SPDT, U1 NCP1117-3.3_SOT223, U10 MomentSwitch, U11 MomentSwitch, U2 STM32F411RETx, U3 lis3dh_board, U4 Pulse_sensor, U5 MAX4460ESA+, U6 Nokia5110, U7 piezo, U8 MomentSwitch, U9 MomentSwitch, Y1 8MHz

Commit message: Hardware finished for ordering
Parts:
- added C20: 100n, Capacitor_SMD:C_0805_2012Metric_Pad1.15x1.40mm_HandSolder, F.Cu at (28.4, 48.2)
- added C21: 100n, Capacitor_SMD:C_0805_2012Metric_Pad1.15x1.40mm_HandSolder, F.Cu at (34.1, 51.0)
- added C22: 100n, Capacitor_SMD:C_0805_2012Metric_Pad1.15x1.40mm_HandSolder, F.Cu at (22.4, 48.2)
- added R18: 1k, Resistor_SMD:R_0805_2012Metric_Pad1.15x1.40mm_HandSolder, F.Cu at (90.7, 45.5)
- moved R15 4.51 mm to (30.5, 52.0), turned to 0 degrees
- moved R17 1.80 mm to (19.7, 48.2)
- moved R2 1.35 mm to (16.9, 48.2), turned to 270 degrees
- moved R16 1.10 mm to (25.9, 48.2)
Connections:
- U4 pad 1: /PULSESIG -> Net-(R18-Pad1)
Routing:
- net /TIM_START: track 48.3 -> 54.8 mm
- net Net-(R18-Pad1): track 0.00 -> 3.50 mm
- net GND: track 31.3 -> 27.8 mm
- net /TIM_INC: track 38.9 -> 41.5 mm
- net /NRST: track 113.7 -> 111.6 mm
- net /TIM_RES: track 32.9 -> 34.7 mm
- net +3V3: track 384.8 -> 384.1 mm
- net /PULSESIG: track 70.3 -> 69.7 mm, vias 1 -> 2
Other:
- board text added: "This side down"
