File: Project/Hardware/Schematic_ons/PCB_Simon_mount_rev2.sch (KiCad schematic (older format))
At the start: 25 parts, among them J1 USB_B_Micro, J2 6P Male, J3 Conn_01x03_Male, SW1 SW_SPDT, U1 NCP1117-3.3_SOT223, U2 STM32F411RETx, Y1 8MHz

Commit message: Add files via upload
Added resistor to pulse, and capacitors to buttons
Parts:
- BT1: symbol Device:Battery -> PCB_Simon_mount_rev2-rescue:Battery-Device
- C1, C10, C11, C12, C13, C14, C15, C2, C3, C4, C5, C6, C7, C8, C9: symbol Device:C_Small -> PCB_Simon_mount_rev2-rescue:C_Small-Device
- J1: symbol Connector:USB_B_Micro -> PCB_Simon_mount_rev2-rescue:USB_B_Micro-Connector
- J2: symbol Connector:Conn_01x06_Male -> PCB_Simon_mount_rev2-rescue:Conn_01x06_Male-Connector
- J3: symbol Connector:Conn_01x03_Male -> PCB_Simon_mount_rev2-rescue:Conn_01x03_Male-Connector
- R1, R2: symbol Device:R_Small -> PCB_Simon_mount_rev2-rescue:R_Small-Device
- SW1: symbol Switch:SW_SPDT -> PCB_Simon_mount_rev2-rescue:SW_SPDT-Switch
- U1: symbol Regulator_Linear:NCP1117-3.3_SOT223 -> PCB_Simon_mount_rev2-rescue:NCP1117-3.3_SOT223-Regulator_Linear
- U2: symbol MCU_ST_STM32F4:STM32F411RETx -> PCB_Simon_mount_rev2-rescue:STM32F411RETx-MCU_ST_STM32F4
- Y1: symbol Device:Crystal -> PCB_Simon_mount_rev2-rescue:Crystal-Device
Changed lines of the file:
@@
 EESchema Schematic File Version 4
+LIBS:PCB_Simon_mount_rev2-cache
 EELAYER 26 0
 EELAYER END
@@
 $EndDescr
 $Comp
-L MCU_ST_STM32F4:STM32F411RETx U2
+L PCB_Simon_mount_rev2-rescue:STM32F411RETx-MCU_ST_STM32F4 U2
 U 1 1 5C49BAEC
 P 6800 4200
@@
 $EndComp
 $Comp
-L Device:C_Small C11
+L PCB_Simon_mount_rev2-rescue:C_Small-Device C11
 U 1 1 5C49BC7E
 P 6400 1300
@@
 $EndComp
 $Comp
-L Device:C_Small C12
+L PCB_Simon_mount_rev2-rescue:C_Small-Device C12
 U 1 1 5C49BCF8
 P 6700 1300
@@
 $EndComp
 $Comp
-L Device:C_Small C13
+L PCB_Simon_mount_rev2-rescue:C_Small-Device C13
 U 1 1 5C49BD16
 P 7000 1300
@@
 $EndComp
 $Comp
-L Device:C_Small C14
+L PCB_Simon_mount_rev2-rescue:C_Small-Device C14
 U 1 1 5C49BD30
 P 7300 1300
@@
 $EndComp
 $Comp
-L Device:C_Small C10
+L PCB_Simon_mount_rev2-rescue:C_Small-Device C10
 U 1 1 5C49BD4E
 P 6100 1300
@@
 $EndComp
 $Comp
-L power:+3V3 #PWR0101
+L PCB_Simon_mount_rev2-rescue:+3V3-power #PWR0101
 U 1 1 5C49BD99
 P 6100 1000
@@
 $EndComp
 $Comp
-L power:GND #PWR0102
+L PCB_Simon_mount_rev2-rescue:GND-power #PWR0102
 U 1 1 5C49BDDC
 P 6100 1600
@@
 	7000 1500 6700 1500
 $Comp
-L power:+3V3 #PWR0103
+L PCB_Simon_mount_rev2-rescue:+3V3-power #PWR0103
 U 1 1 5C49C6AF
 P 6800 2300
@@
 Connection ~ 7000 2400
 $Comp
-L power:GND #PWR0104
+L PCB_Simon_mount_rev2-rescue:GND-power #PWR0104
 U 1 1 5C49DB13
 P 6800 6200
@@
 	6800 6100 6800 6200
 $Comp
-L Device:C_Small C8
+L PCB_Simon_mount_rev2-rescue:C_Small-Device C8
 U 1 1 5C49FE02
 P 5800 1300
@@
 	5800 1500 6100 1500
 $Comp
-L Device:C_Small C9
+L PCB_Simon_mount_rev2-rescue:C_Small-Device C9
 U 1 1 5C4A8076
 P 5900 3100
@@
 $EndComp
 $Comp
-L power:GND #PWR0105
+L PCB_Simon_mount_rev2-rescue:GND-power #PWR0105
 U 1 1 5C4A893E
 P 5600 3200
@@
 Connection ~ 6700 2400
 $Comp
-L Device:R_Small R2
+L PCB_Simon_mount_rev2-rescue:R_Small-Device R2
 U 1 1 5C4AD49E
 P 6000 2500
@@
 $EndComp
 $Comp
-L power:+3V3 #PWR0106
+L PCB_Simon_mount_rev2-rescue:+3V3-power #PWR0106
 U 1 1 5C4AD51D
 P 6000 2300
@@
 	6000 2300 6000 2400
 $Comp
-L Device:R_Small R1
+L PCB_Simon_mount_rev2-rescue:R_Small-Device R1
 U 1 1 5C4AF9C4
 P 5900 2900
@@
 $EndComp
 $Comp
-L Device:Crystal Y1
+L PCB_Simon_mount_rev2-rescue:Crystal-Device Y1
 U 1 1 5C4B6BEC
 P 5600 4000
@@
 	6000 4200 5600 4200
 $Comp
-L Device:C_Small C6
+L PCB_Simon_mount_rev2-rescue:C_Small-Device C6
 U 1 1 5C4C9EDF
 P 5400 3800
@@
 $EndComp
 $Comp
-L Device:C_Small C7
+L PCB_Simon_mount_rev2-rescue:C_Small-Device C7
 U 1 1 5C4C9F37
 P 5400 4200
@@
 Connection ~ 5600 3800
 $Comp
-L power:GND #PWR0107
+L PCB_Simon_mount_rev2-rescue:GND-power #PWR0107
 U 1 1 5C4CB08E
 P 5200 4300
@@
 Connection ~ 5600 4200
 $Comp
-L Connector:Conn_01x06_Male J2
+L PCB_Simon_mount_rev2-rescue:Conn_01x06_Male-Connector J2
 U 1 1 5C4D1603
 P 1400 4400
@@
 SWO
 $Comp
-L power:GND #PWR0108
+L PCB_Simon_mount_rev2-rescue:GND-power #PWR0108
 U 1 1 5C4DD1C0
 P 2700 4800
@@
 	2700 4500 2700 4600
 $Comp
-L power:+3V3 #PWR0109
+L PCB_Simon_mount_rev2-rescue:+3V3-power #PWR0109
 U 1 1 5C4E23FA
 P 2700 4100
@@
 	2700 4100 2700 4200
 $Comp
-L Device:C_Small C3
+L PCB_Simon_mount_rev2-rescue:C_Small-Device C3
 U 1 1 5C4E5BA4
 P 2700 4400
@@
 NoConn ~ 6100 4100
 $Comp
-L Device:C_Small C15
+L PCB_Simon_mount_rev2-rescue:C_Small-Device C15
 U 1 1 5C6BB510
 P 7600 1300
@@
 $EndSheet
 $Comp
-L Device:C_Small C1
+L PCB_Simon_mount_rev2-rescue:C_Small-Device C1
 U 1 1 5C5CED5E
 P 2200 2700
@@
 	2200 2500 2500 2500
 $Comp
-L Device:C_Small C4
+L PCB_Simon_mount_rev2-rescue:C_Small-Device C4
 U 1 1 5C5CED70
 P 3700 2700
@@
 	3700 2800 3700 3000
 $Comp
-L Device:C_Small C5
+L PCB_Simon_mount_rev2-rescue:C_Small-Device C5
 U 1 1 5C5CED79
 P 4000 2700
@@
 $EndComp
 $Comp
-L Device:C_Small C2
+L PCB_Simon_mount_rev2-rescue:C_Small-Device C2
 U 1 1 5C5CED80
 P 2500 2700
@@
 	2200 2300 2200 2500
 $Comp
-L power:+3V3 #PWR0110
+L PCB_Simon_mount_rev2-rescue:+3V3-power #PWR0110
 U 1 1 5C5CED9E
 P 4000 2300
@@
 Connection ~ 4000 2500
 $Comp
-L Regulator_Linear:NCP1117-3.3_SOT223 U1
+L PCB_Simon_mount_rev2-rescue:NCP1117-3.3_SOT223-Regulator_Linear U1
 U 1 1 5C5D379C
 P 3100 2500
@@
 Connection ~ 3700 3000
 $Comp
-L power:GND #PWR0111
+L PCB_Simon_mount_rev2-rescue:GND-power #PWR0111
 U 1 1 5C61536D
 P 3100 3100
@@
 	4000 3000 4000 2800
 $Comp
-L Device:Battery BT1
+L PCB_Simon_mount_rev2-rescue:Battery-Device BT1
 U 1 1 5C624D2E
 P 1200 1300
@@
 $EndComp
 $Comp
-L power:GND #PWR0112
+L PCB_Simon_mount_rev2-rescue:GND-power #PWR0112
 U 1 1 5C6250C7
 P 1200 1700
@@
 $EndComp
 $Comp
-L power:+BATT #PWR0113
+L PCB_Simon_mount_rev2-rescue:+BATT-power #PWR0113
 U 1 1 5C6251FB
 P 1200 900
@@
 TEMPOUT
 $Comp
-L Connector:Conn_01x03_Male J3
+L PCB_Simon_mount_rev2-rescue:Conn_01x03_Male-Connector J3
 U 1 1 5C5B0DFA
 P 1400 5200
@@
 USART1_RX
 $Comp
-L Connector:USB_B_Micro J1
+L PCB_Simon_mount_rev2-rescue:USB_B_Micro-Connector J1
 U 1 1 5C5CFFB9
 P 1150 2700
@@
 	1450 2500 1600 2500
 $Comp
-L power:+5V #PWR0114
+L PCB_Simon_mount_rev2-rescue:+5V-power #PWR0114
 U 1 1 5C5E52AC
 P 1600 2500
@@
 Data-
 $Comp
-L power:GND #PWR0115
+L PCB_Simon_mount_rev2-rescue:GND-power #PWR0115
 U 1 1 5C5E53D4
 P 1150 3100
@@
 NoConn ~ 1450 2800
 $Comp
-L Switch:SW_SPDT SW1
+L PCB_Simon_mount_rev2-rescue:SW_SPDT-Switch SW1
 U 1 1 5C6D5462
 P 3000 1400
@@
 	3300 1400 3200 1400
 $Comp
-L power:+BATT #PWR0117
+L PCB_Simon_mount_rev2-rescue:+BATT-power #PWR0117
 U 1 1 5C6F447A
 P 2500 1100
@@
 	2500 1300 2500 1100
 $Comp
-L power:+5V #PWR0118
+L PCB_Simon_mount_rev2-rescue:+5V-power #PWR0118
 U 1 1 5C6FA90C
 P 2300 1400

Commit message: Hardware finished for ordering
Parts:
- J1: footprint PASC1:USB_Micro_B_Female_10118193-0001LF -> PASC:USB_Micro_B_Female_10118193-0001LF
Changed lines of the file:
@@
 F 0 "J1" H 1205 3167 50  0000 C CNN
 F 1 "USB_B_Micro" H 1205 3076 50  0000 C CNN
-F 2 "PASC1:USB_Micro_B_Female_10118193-0001LF" H 1300 2650 50  0001 C CNN
+F 2 "PASC:USB_Micro_B_Female_10118193-0001LF" H 1300 2650 50  0001 C CNN
 F 3 "~" H 1300 2650 50  0001 C CNN
 	1    1150 2700
