File: Project/Hardware/Schematic_ons/buttons.sch (KiCad schematic (older format))
At the start: 7 parts, among them U10 MomentSwitch, U11 MomentSwitch, U8 MomentSwitch, U9 MomentSwitch

Commit message: Pcb rev1 simon (#14)
Klar PCB av Simon
Added resistor to pulse, and capacitors to buttons
Parts:
- added C20, C21, C22: 100n, Capacitors_SMD:C_0805_HandSoldering, symbol Device:C_Small
- R15, R16, R17: symbol Device:R -> PCB_Simon_mount_rev2-rescue:R-Device
Connections:
- net GND: now also C20.2, C21.2, C22.2
- net TIM_INC: now also C20.1
- net TIM_RES: now also C22.1
- net TIM_START: now also C21.1
Changed lines of the file:
@@
 EESchema Schematic File Version 4
-LIBS:lab-cache
+LIBS:PCB_Simon_mount_rev2-cache
 EELAYER 26 0
 EELAYER END
@@
 	2250 1400 2250 1600
 $Comp
-L power:GND #PWR0139
+L PCB_Simon_mount_rev2-rescue:GND-power #PWR0139
 U 1 1 5C5ED863
 P 2150 1400
@@
 	2250 3000 2250 3200
 $Comp
-L power:+3.3V #PWR0140
+L PCB_Simon_mount_rev2-rescue:+3.3V-power #PWR0140
 U 1 1 5C68E9D0
 P 2050 3100
@@
 	3150 3000 3150 3200
 $Comp
-L Device:R R15
+L PCB_Simon_mount_rev2-rescue:R-Device R15
 U 1 1 5C68EFD4
 P 3450 3550
@@
 	3150 3200 3150 3400
 $Comp
-L power:GND #PWR0141
+L PCB_Simon_mount_rev2-rescue:GND-power #PWR0141
 U 1 1 5C68F32C
 P 3450 3800
@@
 $EndComp
 Wire Wire Line
-	3450 3700 3450 3800
+	3450 3700 3450 3750
 Wire Wire Line
 	3450 3400 3450 3200
 Connection ~ 3450 3200
 Wire Wire Line
-	3450 3200 3650 3200
+	3450 3200 3600 3200
 $Comp
 L PASC:MomentSwitch U10
@@
 	2250 4350 2250 4550
 $Comp
-L power:+3.3V #PWR0142
+L PCB_Simon_mount_rev2-rescue:+3.3V-power #PWR0142
 U 1 1 5C68FAC8
 P 2050 4450
@@
 	3150 4350 3150 4550
 $Comp
-L Device:R R16
+L PCB_Simon_mount_rev2-rescue:R-Device R16
 U 1 1 5C68FAD3
 P 3450 4900
@@
 	3150 4550 3150 4750
 $Comp
-L power:GND #PWR0143
+L PCB_Simon_mount_rev2-rescue:GND-power #PWR0143
 U 1 1 5C68FADD
 P 3450 5150
@@
 $EndComp
 Wire Wire Line
-	3450 5050 3450 5150
+	3450 5050 3450 5100
 Wire Wire Line
 	3450 4750 3450 4550
 Connection ~ 3450 4550
 Wire Wire Line
-	3450 4550 3650 4550
+	3450 4550 3550 4550
 $Comp
 L PASC:MomentSwitch U11
@@
 	2250 5550 2250 5750
 $Comp
-L power:+3.3V #PWR0144
+L PCB_Simon_mount_rev2-rescue:+3.3V-power #PWR0144
 U 1 1 5C6902FE
 P 2050 5650
@@
 	3150 5550 3150 5750
 $Comp
-L Device:R R17
+L PCB_Simon_mount_rev2-rescue:R-Device R17
 U 1 1 5C690309
 P 3450 6100
@@
 	3150 5750 3150 5950
 $Comp
-L power:GND #PWR0145
+L PCB_Simon_mount_rev2-rescue:GND-power #PWR0145
 U 1 1 5C690313
 P 3450 6350
@@
 $EndComp
 Wire Wire Line
-	3450 6250 3450 6350
+	3450 6250 3450 6300
 Wire Wire Line
 	3450 5950 3450 5750
 Connection ~ 3450 5750
 Wire Wire Line
-	3450 5750 3650 5750
+	3450 5750 3550 5750
+$Comp
+L Device:C_Small C21
+U 1 1 5C6871FB
+P 3700 3550
+F 0 "C21" H 3792 3596 50  0000 L CNN
+F 1 "100n" H 3792 3505 50  0000 L CNN
+F 2 "Capacitors_SMD:C_0805_HandSoldering" H 3700 3550 50  0001 C CNN
+F 3 "~" H 3700 3550 50  0001 C CNN
+	1    3700 3550
+	1    0    0    -1
+$EndComp
+$Comp
+L Device:C_Small C20
+U 1 1 5C687354
+P 3650 4900
+F 0 "C20" H 3742 4946 50  0000 L CNN
+F 1 "100n" H 3742 4855 50  0000 L CNN
+F 2 "Capacitors_SMD:C_0805_HandSoldering" H 3650 4900 50  0001 C CNN
+F 3 "~" H 3650 4900 50  0001 C CNN
+	1    3650 4900
+	1    0    0    -1
+$EndComp
+$Comp
+L Device:C_Small C22
+U 1 1 5C687D78
+P 3700 6100
+F 0 "C22" H 3792 6146 50  0000 L CNN
+F 1 "100n" H 3792 6055 50  0000 L CNN
+F 2 "Capacitors_SMD:C_0805_HandSoldering" H 3700 6100 50  0001 C CNN
+F 3 "~" H 3700 6100 50  0001 C CNN
+	1    3700 6100
+	1    0    0    -1
+$EndComp
+Wire Wire Line
+	3650 5000 3650 5100
+Wire Wire Line
+	3650 5100 3450 5100
+Connection ~ 3450 5100
+Wire Wire Line
+	3450 5100 3450 5150
+Wire Wire Line
+	3650 4800 3650 4650
+Wire Wire Line
+	3650 4650 3550 4650
+Wire Wire Line
+	3550 4650 3550 4550
+Connection ~ 3550 4550
+Wire Wire Line
+	3550 4550 3650 4550
+Wire Wire Line
+	3700 3650 3700 3750
+Wire Wire Line
+	3700 3750 3450 3750
+Connection ~ 3450 3750
+Wire Wire Line
+	3450 3750 3450 3800
+Wire Wire Line
+	3700 3450 3600 3450
+Wire Wire Line
+	3600 3450 3600 3200
+Connection ~ 3600 3200
+Wire Wire Line
+	3600 3200 3650 3200
+Wire Wire Line
+	3700 6200 3700 6300
+Wire Wire Line
+	3700 6300 3450 6300
+Connection ~ 3450 6300
+Wire Wire Line
+	3450 6300 3450 6350
+Wire Wire Line
+	3700 6000 3700 5850
+Wire Wire Line
+	3700 5850 3550 5850
+Wire Wire Line
+	3550 5850 3550 5750
+Connection ~ 3550 5750
+Wire Wire Line
+	3550 5750 3650 5750
 $EndSCHEMATC

Commit message: Hardware finished for ordering
Parts:
- C20, C21, C22: footprint Capacitors_SMD:C_0805_HandSoldering -> Capacitor_SMD:C_0805_2012Metric_Pad1.15x1.40mm_HandSolder
Changed lines of the file:
@@
 F 0 "C21" H 3792 3596 50  0000 L CNN
 F 1 "100n" H 3792 3505 50  0000 L CNN
-F 2 "Capacitors_SMD:C_0805_HandSoldering" H 3700 3550 50  0001 C CNN
+F 2 "Capacitor_SMD:C_0805_2012Metric_Pad1.15x1.40mm_HandSolder" H 3700 3550 50  0001 C CNN
 F 3 "~" H 3700 3550 50  0001 C CNN
 	1    3700 3550
@@
 F 0 "C20" H 3742 4946 50  0000 L CNN
 F 1 "100n" H 3742 4855 50  0000 L CNN
-F 2 "Capacitors_SMD:C_0805_HandSoldering" H 3650 4900 50  0001 C CNN
+F 2 "Capacitor_SMD:C_0805_2012Metric_Pad1.15x1.40mm_HandSolder" H 3650 4900 50  0001 C CNN
 F 3 "~" H 3650 4900 50  0001 C CNN
 	1    3650 4900
@@
 F 0 "C22" H 3792 6146 50  0000 L CNN
 F 1 "100n" H 3792 6055 50  0000 L CNN
-F 2 "Capacitors_SMD:C_0805_HandSoldering" H 3700 6100 50  0001 C CNN
+F 2 "Capacitor_SMD:C_0805_2012Metric_Pad1.15x1.40mm_HandSolder" H 3700 6100 50  0001 C CNN
 F 3 "~" H 3700 6100 50  0001 C CNN
 	1    3700 6100
