File: Project/Hardware/Schematic_ons/pulsesensor.sch (KiCad schematic (older format))
At the start: 2 parts, among them U4 Pulse_sensor

Commit message: Add files via upload
Added resistor to pulse, and capacitors to buttons
Parts:
- added R18: 1k, Resistors_SMD:R_0805_HandSoldering, symbol Device:R
- C17: symbol Device:C -> PCB_Simon_mount_rev2-rescue:C-Device
Connections:
- net PULSESIG: now also R18.2; no longer U4.1 (Signal)
- new net: R18.1, U4.1 (Signal)
Changed lines of the file:
@@
 EESchema Schematic File Version 4
+LIBS:PCB_Simon_mount_rev2-cache
 EELAYER 26 0
 EELAYER END
@@
 $EndComp
 $Comp
-L power:+3V3 #PWR0125
+L PCB_Simon_mount_rev2-rescue:+3V3-power #PWR0125
 U 1 1 5C5DA797
 P 3400 1500
@@
 $EndComp
 $Comp
-L Device:C C17
+L PCB_Simon_mount_rev2-rescue:C-Device C17
 U 1 1 5C5DA7DA
 P 3250 2100
@@
 	3400 1800 3400 1500
 $Comp
-L power:GND #PWR0126
+L PCB_Simon_mount_rev2-rescue:GND-power #PWR0126
 U 1 1 5C5DA906
 P 2400 2550
@@
 $EndComp
 $Comp
-L power:GND #PWR0127
+L PCB_Simon_mount_rev2-rescue:GND-power #PWR0127
 U 1 1 5C5DA96D
 P 3250 2600
@@
 Wire Wire Line
 	2400 2300 2400 2550
-Text HLabel 1950 1800 0    50   Input ~ 0
+Text HLabel 1100 1800 0    50   Input ~ 0
 PULSESIG
+$Comp
+L Device:R R18
+U 1 1 5C68650D
+P 1350 1800
+F 0 "R18" V 1143 1800 50  0000 C CNN
+F 1 "1k" V 1234 1800 50  0000 C CNN
+F 2 "Resistors_SMD:R_0805_HandSoldering" V 1280 1800 50  0001 C CNN
+F 3 "~" H 1350 1800 50  0001 C CNN
+	1    1350 1800
+	0    1    1    0
+$EndComp
+Wire Wire Line
+	1500 1800 1950 1800
+Wire Wire Line
+	1200 1800 1100 1800
 $EndSCHEMATC

Commit message: Hardware finished for ordering
Parts:
- R18: footprint Resistors_SMD:R_0805_HandSoldering -> Resistor_SMD:R_0805_2012Metric_Pad1.15x1.40mm_HandSolder
Changed lines of the file:
@@
 Wire Wire Line
 	2400 2300 2400 2550
-Text HLabel 1100 1800 0    50   Input ~ 0
-PULSESIG
+Wire Wire Line
+	1950 1800 1500 1800
+Wire Wire Line
+	1200 1800 1100 1800
 $Comp
 L Device:R R18
@@
 F 0 "R18" V 1143 1800 50  0000 C CNN
 F 1 "1k" V 1234 1800 50  0000 C CNN
-F 2 "Resistors_SMD:R_0805_HandSoldering" V 1280 1800 50  0001 C CNN
+F 2 "Resistor_SMD:R_0805_2012Metric_Pad1.15x1.40mm_HandSolder" V 1280 1800 50  0001 C CNN
 F 3 "~" H 1350 1800 50  0001 C CNN
 	1    1350 1800
 	0    1    1    0
 $EndComp
-Wire Wire Line
-	1500 1800 1950 1800
-Wire Wire Line
-	1200 1800 1100 1800
+Text HLabel 1100 1800 0    50   Input ~ 0
+PULSESIG
 $EndSCHEMATC
